Commit message: feat: update wheel physics to 10-inch specs and add mesh assets

File: src/mona_description/urdf/mona.urdf.xacro (robot description, xacro)
@@ -1,19 +1,23 @@
 <?xml version="1.0"?>
 <robot xmlns:xacro="http://www.ros.org/wiki/xacro" name="mona">
-    <xacro:property name="base_length"    value="1.25"/>
-    <xacro:property name="base_width"     value="0.8"/>
-    <xacro:property name="base_height"    value="0.3"/>
-    <xacro:property name="base_mass"      value="150.0"/>
-    <xacro:property name="wheel_radius"   value="0.1"/>
-    <xacro:property name="wheel_width"    value="0.08"/>
-    <xacro:property name="wheel_mass"     value="5.0"/>
-    <xacro:property name="wheel_x_offset" value="0.40"/>
-    <xacro:property name="wheel_y_offset" value="0.40"/>
-    <xacro:property name="wheel_z_offset" value="-0.15"/>
+    <xacro:property name="base_length"  value="1.25"/>
+    <xacro:property name="base_width"   value="0.80"/>
+    <xacro:property name="base_height"  value="0.30"/>
+    <xacro:property name="base_mass"    value="150.0"/>
+    <xacro:property name="robot_road_clearance" value="0.02"/>
+    <xacro:property name="wheel_radius" value="0.127"/>
+    <xacro:property name="wheel_width"  value="0.10"/>
+    <xacro:property name="wheel_mass"   value="15.0"/>
+    <xacro:property name="wheel_base_x" value="${0.8 / 2}"/>
+    <xacro:property name="wheel_base_y" value="${base_width/2 + wheel_width/2 + 0.002}"/>
+    <xacro:property name="wheel_base_z" value="${-base_height/2 - robot_road_clearance + wheel_radius}"/>
+    <xacro:property name="robot_spawn_x" value="0.0"/>
+    <xacro:property name="robot_spawn_y" value="0.0"/>
+    <xacro:property name="robot_spawn_z" value="${(robot_road_clearance+0.003) + (base_height/2)}"/>
     <link name="base_footprint"/>
     <joint name="base_joint" type="fixed">
         <parent link="base_footprint"/>
         <child link="base_link"/>
-        <origin xyz="0 0 ${base_height/2.0 + 0.02}" rpy="0 0 0"/>
+        <origin xyz="${robot_spawn_x} ${robot_spawn_y} ${robot_spawn_z}" rpy="0 0 0"/>
     </joint>
     <link name="base_link">
@@ -44,8 +48,7 @@
         <link name="${name}_link">
             <visual>
-                <origin xyz="0 0 0" rpy="${pi/2} 0 0"/>
-                <geometry>
+                <origin xyz="0 0 0" rpy="${pi/2} 0 0"/> <geometry>
                     <cylinder radius="${wheel_radius}" length="${wheel_width}"/>
-                </geometry>
+                    </geometry>
                 <material name="black">
                     <color rgba="0.1 0.1 0.1 1.0"/>
@@ -69,17 +72,17 @@
             <parent link="base_link"/>
             <child link="${name}_link"/>
-            <origin xyz="${x} ${y} ${wheel_z_offset}" rpy="0 0 0"/>
+            <origin xyz="${x} ${y} ${wheel_base_z}" rpy="0 0 0"/>
             <axis xyz="0 1 0"/>
         </joint>
         <gazebo reference="${name}_link">
-            <material>Gazebo/Black</material>
+            <material>Gazebo/Grey</material>
             <mu1>0.8</mu1>
             <mu2>0.8</mu2>
         </gazebo>
     </xacro:macro>
-    <xacro:mecanum_wheel name="front_left_wheel"  x="${wheel_x_offset}"  y="${wheel_y_offset}"  flip_visual="1"/>
-    <xacro:mecanum_wheel name="front_right_wheel" x="${wheel_x_offset}"  y="-${wheel_y_offset}" flip_visual="0"/>
-    <xacro:mecanum_wheel name="rear_left_wheel"   x="-${wheel_x_offset}" y="${wheel_y_offset}"  flip_visual="1"/>
-    <xacro:mecanum_wheel name="rear_right_wheel"  x="-${wheel_x_offset}" y="-${wheel_y_offset}" flip_visual="0"/>
+    <xacro:mecanum_wheel name="wheel_front_left"  x="${wheel_base_x}"  y="${wheel_base_y}"  flip_visual="1"/>
+    <xacro:mecanum_wheel name="wheel_rear_left"   x="-${wheel_base_x}" y="${wheel_base_y}"  flip_visual="1"/>
+    <xacro:mecanum_wheel name="wheel_front_right" x="${wheel_base_x}"  y="-${wheel_base_y}" flip_visual="-1"/>
+    <xacro:mecanum_wheel name="wheel_rear_right"  x="-${wheel_base_x}" y="-${wheel_base_y}" flip_visual="-1"/>
     <gazebo>
         <plugin name="object_controller" filename="libgazebo_ros_planar_move.so">
